File: hardware/kicad/rools-core/rools-core.kicad_pcb (KiCad board)
At the start: 4 copper layers, 102 x 108 mm, 148 parts, among them J1 EURO_PWR, J2 EXP_BUS, J4 ST7789, J6 J_TOP_UI, J7 J_TOP_MAIN, SW1 RotaryEncoder_Switch, SW2 RotaryEncoder_Switch, SW3 SW_Push, U1 AP2112K-3.3, U10 LM393, U2 TPS54302, U4 OPA4171, U5 MCP6004, U6 LM4040DBZ-10, U7 TL074, U8 TL074, U9 DAC8565

Commit message: Continue Core PCB routing and tune board design rules.
Fix seed debug header to 1x10 and add preset track/via widths for layout work.

Co-authored-by: Cursor <cursoragent@cursor.com>
Parts:
- C21, C22, C23, C24, C25, C26, C27, C28, C29, C30, C31, C32, C9, R3, R4, R44, R45, R46, R47, R48, R49, R50, R51, R52, R53, R54, R55, R56, R57, R58, R59, R60, R61, R62, R63, U7, U8: moved to F.Cu
- J_BM_R1: footprint Connector_PinSocket_2.54mm:PinSocket_1x11_P2.54mm_Vertical -> Connector_PinSocket_2.54mm:PinSocket_1x10_P2.54mm_Vertical
- R21, R22: moved to B.Cu
- moved R7 111.3 mm to (162.7, 57.2), turned to 180 degrees
- moved R10 109.4 mm to (157.1, 59.0), turned to 0 degrees
- moved R9 108.4 mm to (157.1, 57.2), turned to 0 degrees
- moved R15 107.7 mm to (162.7, 60.5), turned to 0 degrees
- moved R8 107.4 mm to (162.7, 58.9)
- moved C12 105.6 mm to (159.8, 59.5), turned to -90 degrees
- moved R16 104.7 mm to (157.1, 60.7), turned to 180 degrees
- moved U4 96.9 mm to (159.8, 65.8), turned to -90 degrees
- moved R19 95.3 mm to (158.9, 78.3), turned to -90 degrees
- moved C15 92.4 mm to (186.8, 63.5), turned to 180 degrees
- moved R18 91.1 mm to (162.7, 71.0), turned to 0 degrees
- moved R20 90.8 mm to (157.2, 78.3)
- moved R32 90.0 mm to (186.8, 65.2), turned to 180 degrees
- moved R25 89.7 mm to (189.1, 61.9), turned to -90 degrees
- moved C13 89.7 mm to (159.8, 71.8)
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Routing:
- net +3V3_A: track 133.6 -> 0.20 mm, vias 2 -> 0
- net +5V: track 110.5 -> 34.2 mm, vias 1 -> 3
- net +12V: track 28.7 -> 104.4 mm, vias 3 -> 5
- net -12V: track 23.1 -> 98.6 mm, vias 4 -> 5
- net EXP_GPIO0: track 64.6 -> 0.00 mm
- net GND: track 118.4 -> 58.0 mm, vias 26 -> 15
- net J_CV_IN_1: track 52.3 -> 0.00 mm
- net J_CV_IN_2: track 52.0 -> 0.00 mm
- net +3V3_DAC: track 30.0 -> 75.4 mm
- net J_CV_IN_4: track 35.7 -> 0.00 mm
- net AUDIO_IN_R: track 0.00 -> 34.2 mm, vias 0 -> 1
- net USB_D+: track 33.5 -> 0.00 mm
- net USB_D-: track 32.5 -> 0.00 mm
- net J_CV_IN_3: track 31.9 -> 0.00 mm
- net I2C_SDA: track 31.0 -> 0.00 mm, vias 1 -> 0
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