File: hardware/kicad/rools-core/sheets/seed.kicad_sch (KiCad schematic)
At the start: 5 parts, among them J2 EXP_BUS, J7 J_TOP_MAIN

Commit message: Continue Core PCB routing and tune board design rules.
Fix seed debug header to 1x10 and add preset track/via widths for layout work.

Co-authored-by: Cursor <cursoragent@cursor.com>
Parts:
- J_BM_R1: footprint Connector_PinSocket_2.54mm:PinSocket_1x11_P2.54mm_Vertical -> Connector_PinSocket_2.54mm:PinSocket_1x10_P2.54mm_Vertical
Changed lines of the file:
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@@
 			)
 		)
-		(property "Footprint" "Connector_PinSocket_2.54mm:PinSocket_1x11_P2.54mm_Vertical"
+		(property "Footprint" "Connector_PinSocket_2.54mm:PinSocket_1x10_P2.54mm_Vertical"
 			(at 116.84 130.81 0)
 			(hide yes)
